Commit message: Add gripper frames.

File: romeo_description/urdf/romeo.urdf (robot description, URDF)
Before this commit: robot romeo, 68 links, 67 joints
Links:
- added link l_gripper
- added link r_gripper
Joints:
- added joint l_gripper_joint: type fixed, parent l_wrist, child l_gripper, origin xyz=0.09 0 -0.02 rpy=1.57079633 0 0
- added joint r_gripper_joint: type fixed, parent r_wrist, child r_gripper, origin xyz=0.09 0 -0.02 rpy=-1.57079633 0 0

File: romeo_description/urdf/romeo_small.urdf (robot description, URDF)
Before this commit: robot romeo, 44 links, 43 joints
Links:
- added link l_gripper
- added link r_gripper
Joints:
- added joint l_gripper_joint: type fixed, parent l_wrist, child l_gripper, origin xyz=0.09 0 -0.02 rpy=1.57079633 0 0
- added joint r_gripper_joint: type fixed, parent r_wrist, child r_gripper, origin xyz=0.09 0 -0.02 rpy=1.57079633 0 0
